Commit message: 👌 IMPROVE: Errors fixed and meshes implemented

File: cefiro_sensors/urdf/imu_icm42670p/imu_icm42670p.urdf.xacro (robot description, xacro)
@@ -1,9 +1,9 @@
 <?xml version="1.0"?>
-<robot name="bmp581"
+<robot name="imu_icm42670p"
     xmlns:xacro="http://www.ros.org/wiki/xacro">
     <!-- Load physical & visual parameters -->
     <xacro:arg name="physical_config_file" default="$(find cefiro_sensors)/config/imu_icm42670p.yaml"/>
     <xacro:property name="L" value="${xacro.load_yaml('$(arg physical_config_file)')['imu_icm42670p']['base_link']}"/>
-    <xacro:property name="mesh_dir" value="package://cefiro_sensors/urdf/bmp581/meshes"/>
+    <xacro:property name="mesh_dir" value="package://cefiro_sensors/urdf/imu_icm42670p/meshes"/>
     <!-- Unit conversions -->
     <xacro:property name="g_to_kg" value="${0.001}"/>
@@ -15,5 +15,5 @@
             <origin xyz="${L['visual_origin_xyz'][0]} ${L['visual_origin_xyz'][1]} ${L['visual_origin_xyz'][2]}" rpy="${L['visual_origin_rpy'][0]} ${L['visual_origin_rpy'][1]} ${L['visual_origin_rpy'][2]}" />
             <geometry>
-                <mesh filename="${mesh_dir}/visuals/base_link.stl" scale="1.0 1.0 1.0"/>
+                <mesh filename="${mesh_dir}/base_link.stl" scale="1.0 1.0 1.0"/>
             </geometry>
         </visual>
@@ -31,4 +31,4 @@
     </link>
     <!-- Includes gz model configuration for sim -->
-    <xacro:include filename="$(find cefiro_sensors)/urdf/imu_icm42670p/imu_icm42670p_gz.xacro"/>
+    <xacro:include filename="$(find cefiro_sensors)/urdf/imu_icm42670p/imu_icm42670p_gz.urdf.xacro"/>
 </robot>

File: cefiro_sensors/urdf/magnetometer_mmc5983ma/magnetometer_mmc5983ma.urdf.xacro (robot description, xacro)
@@ -1,9 +1,9 @@
 <?xml version="1.0"?>
-<robot name="bmp581"
+<robot name="magnetometer_mmc5983ma"
     xmlns:xacro="http://www.ros.org/wiki/xacro">
     <!-- Load physical & visual parameters -->
     <xacro:arg name="physical_config_file" default="$(find cefiro_sensors)/config/magnetometer_mmc5983ma.yaml"/>
     <xacro:property name="L" value="${xacro.load_yaml('$(arg physical_config_file)')['magnetometer_mmc5983ma']['base_link']}"/>
-    <xacro:property name="mesh_dir" value="package://cefiro_sensors/urdf/bmp581/meshes"/>
+    <xacro:property name="mesh_dir" value="package://cefiro_sensors/urdf/magnetometer_mmc5983ma/meshes"/>
     <!-- Unit conversions -->
     <xacro:property name="g_to_kg" value="${0.001}"/>
@@ -15,5 +15,5 @@
             <origin xyz="${L['visual_origin_xyz'][0]} ${L['visual_origin_xyz'][1]} ${L['visual_origin_xyz'][2]}" rpy="${L['visual_origin_rpy'][0]} ${L['visual_origin_rpy'][1]} ${L['visual_origin_rpy'][2]}" />
             <geometry>
-                <mesh filename="${mesh_dir}/visuals/base_link.stl" scale="1.0 1.0 1.0"/>
+                <mesh filename="${mesh_dir}/base_link.stl" scale="1.0 1.0 1.0"/>
             </geometry>
         </visual>
