Commit message: ✨ New Feature: RViz2 visualization available for CEFIRO's frame, gyro and their assembly

File: cefiro_description/urdf/cefiro.xacro (robot description, xacro)
@@ -2,6 +2,5 @@
 <robot name="cefiro"
   xmlns:xacro="http://www.ros.org/wiki/xacro">
-  <xacro:include filename="$(find cefiro_description)/urdf/materials.xacro" />
-  <link name="base_link">
+  <link name="chassis_lower_plate">
     <inertial>
       <origin xyz="0.0490073468858582 0.03543104743409582 0.0015000000000000005" rpy="0 0 0"/>
@@ -12,5 +11,5 @@
       <origin xyz="0 0 0" rpy="0 0 0"/>
       <geometry>
-        <mesh filename="package://cefiro_description/meshes/base_link.stl" scale="0.001 0.001 0.001"/>
+        <mesh filename="package://cefiro_description/meshes/frame/chassis_lower_plate.stl" scale="0.001 0.001 0.001"/>
       </geometry>
       <material name="silver"/>
@@ -19,5 +18,25 @@
       <origin xyz="0 0 0" rpy="0 0 0"/>
       <geometry>
-        <mesh filename="package://cefiro_description/meshes/base_link.stl" scale="0.001 0.001 0.001"/>
+        <mesh filename="package://cefiro_description/meshes/frame/chassis_lower_plate.stl" scale="0.001 0.001 0.001"/>
+      </geometry>
+    </collision>
+  </link>
+  <link name="chassis_upper_plate_1">
+    <inertial>
+      <origin xyz="7.358559962991618e-06 -6.906990589405915e-05 0.0017251406233937646" rpy="0 0 0"/>
+      <mass value="0.0364787939875615"/>
+      <inertia ixx="5.6e-05" iyy="3.3e-05" izz="8.9e-05" ixy="-0.0" iyz="-0.0" ixz="0.0"/>
+    </inertial>
+    <visual>
+      <origin xyz="-0.049 -0.0355 -0.003" rpy="0 0 0"/>
+      <geometry>
+        <mesh filename="package://cefiro_description/meshes/frame/chassis_upper_plate_1.stl" scale="0.001 0.001 0.001"/>
+      </geometry>
+      <material name="silver"/>
+    </visual>
+    <collision>
+      <origin xyz="-0.049 -0.0355 -0.003" rpy="0 0 0"/>
+      <geometry>
+        <mesh filename="package://cefiro_description/meshes/frame/chassis_upper_plate_1.stl" scale="0.001 0.001 0.001"/>
       </geometry>
     </collision>
@@ -25,39 +44,439 @@
   <link name="esc_dummy_1">
     <inertial>
-      <origin xyz="4.871638824011093e-07 2.0816681711721685e-17 0.0029999999999999983" rpy="0 0 0"/>
+      <origin xyz="4.871638824011093e-07 2.0816681711721685e-17 0.0029999999999999975" rpy="0 0 0"/>
       <mass value="0.021245400000000005"/>
       <inertia ixx="3e-06" iyy="3e-06" izz="7e-06" ixy="0.0" iyz="0.0" ixz="0.0"/>
     </inertial>
     <visual>
-      <origin xyz="-0.049 -0.0355 -0.003" rpy="0 0 0"/>
-      <geometry>
-        <mesh filename="package://cefiro_description/meshes/esc_dummy_1.stl" scale="0.001 0.001 0.001"/>
-      </geometry>
-      <material name="silver"/>
-    </visual>
-    <collision>
-      <origin xyz="-0.049 -0.0355 -0.003" rpy="0 0 0"/>
-      <geometry>
-        <mesh filename="package://cefiro_description/meshes/esc_dummy_1.stl" scale="0.001 0.001 0.001"/>
-      </geometry>
-    </collision>
-  </link>
-  <link name="chassis_upper_plate_1">
-    <inertial>
-      <origin xyz="7.017397302376549e-06 -6.564061223595513e-05 0.0017139624799641442" rpy="0 0 0"/>
-      <mass value="0.03838457294189457"/>
-      <inertia ixx="5.7e-05" iyy="3.5e-05" izz="9.3e-05" ixy="-0.0" iyz="-0.0" ixz="0.0"/>
-    </inertial>
-    <visual>
-      <origin xyz="-0.049 -0.0355 -0.009" rpy="0 0 0"/>
-      <geometry>
-        <mesh filename="package://cefiro_description/meshes/chassis_upper_plate_1.stl" scale="0.001 0.001 0.001"/>
-      </geometry>
-      <material name="silver"/>
-    </visual>
-    <collision>
-      <origin xyz="-0.049 -0.0355 -0.009" rpy="0 0 0"/>
-      <geometry>
-        <mesh filename="package://cefiro_description/meshes/chassis_upper_plate_1.stl" scale="0.001 0.001 0.001"/>
+      <origin xyz="-0.049 -0.0355 -0.006" rpy="0 0 0"/>
+      <geometry>
+        <mesh filename="package://cefiro_description/meshes/frame/esc_dummy_1.stl" scale="0.001 0.001 0.001"/>
+      </geometry>
+      <material name="silver"/>
+    </visual>
+    <collision>
+      <origin xyz="-0.049 -0.0355 -0.006" rpy="0 0 0"/>
+      <geometry>
+        <mesh filename="package://cefiro_description/meshes/frame/esc_dummy_1.stl" scale="0.001 0.001 0.001"/>
+      </geometry>
+    </collision>
+  </link>
+  <link name="arm_coupling_1">
+    <inertial>
+      <origin xyz="0.013028210396098056 0.006815018249825843 0.017011481507627036" rpy="0 0 0"/>
+      <mass value="0.0378932947271681"/>
+      <inertia ixx="8e-06" iyy="9e-06" izz="9e-06" ixy="1e-06" iyz="-0.0" ixz="0.0"/>
+    </inertial>
+    <visual>
+      <origin xyz="-0.07068 0.026359 -0.003" rpy="0 0 0"/>
+      <geometry>
+        <mesh filename="package://cefiro_description/meshes/frame/arm_coupling_1.stl" scale="0.001 0.001 0.001"/>
+      </geometry>
+      <material name="silver"/>
+    </visual>
+    <collision>
+      <origin xyz="-0.07068 0.026359 -0.003" rpy="0 0 0"/>
+      <geometry>
+        <mesh filename="package://cefiro_description/meshes/frame/arm_coupling_1.stl" scale="0.001 0.001 0.001"/>
+      </geometry>
+    </collision>
+  </link>
+  <link name="propeller_arm_1">
+    <inertial>
+      <origin xyz="0.024748892864255592 -0.02474877464385651 -3.8163916471489756e-17" rpy="0 0 0"/>
+      <mass value="0.01766678419295193"/>
+      <inertia ixx="5e-06" iyy="5e-06" izz="8e-06" ixy="3e-06" iyz="-0.0" ixz="0.0"/>
+    </inertial>
+    <visual>
+      <origin xyz="-0.09365 0.030467 -0.0198" rpy="0 0 0"/>
+      <geometry>
+        <mesh filename="package://cefiro_description/meshes/frame/propeller_arm_1.stl" scale="0.001 0.001 0.001"/>
+      </geometry>
+      <material name="silver"/>
+    </visual>
+    <collision>
+      <origin xyz="-0.09365 0.030467 -0.0198" rpy="0 0 0"/>
+      <geometry>
+        <mesh filename="package://cefiro_description/meshes/frame/propeller_arm_1.stl" scale="0.001 0.001 0.001"/>
+      </geometry>
+    </collision>
+  </link>
+  <link name="arm-motor_coupling_1">
+    <inertial>
+      <origin xyz="0.005140108724772996 -0.0051399000344490575 4.462910693781019e-09" rpy="0 0 0"/>
+      <mass value="0.17482105870117712"/>
+      <inertia ixx="3.3e-05" iyy="3.3e-05" izz="2.9e-05" ixy="-4e-06" iyz="0.0" ixz="0.0"/>
+    </inertial>
+    <visual>
+      <origin xyz="-0.143148 0.079965 -0.0198" rpy="0 0 0"/>
+      <geometry>
+        <mesh filename="package://cefiro_description/meshes/frame/arm-motor_coupling_1.stl" scale="0.001 0.001 0.001"/>
+      </geometry>
+      <material name="silver"/>
+    </visual>
+    <collision>
+      <origin xyz="-0.143148 0.079965 -0.0198" rpy="0 0 0"/>
+      <geometry>
+        <mesh filename="package://cefiro_description/meshes/frame/arm-motor_coupling_1.stl" scale="0.001 0.001 0.001"/>
+      </geometry>
+    </collision>
+  </link>
+  <link name="motor_coupling_1">
+    <inertial>
+      <origin xyz="0.024735903341897042 -0.024978176445044395 0.003012980980874616" rpy="0 0 0"/>
+      <mass value="0.08266534784043636"/>
+      <inertia ixx="3.7e-05" iyy="3.8e-05" izz="4.7e-05" ixy="1.1e-05" iyz="6e-06" ixz="-6e-06"/>
+    </inertial>
+    <visual>
+      <origin xyz="-0.15729 0.094107 -0.0198" rpy="0 0 0"/>
+      <geometry>
+        <mesh filename="package://cefiro_description/meshes/frame/motor_coupling_1.stl" scale="0.001 0.001 0.001"/>
+      </geometry>
+      <material name="silver"/>
+    </visual>
+    <collision>
+      <origin xyz="-0.15729 0.094107 -0.0198" rpy="0 0 0"/>
+      <geometry>
+        <mesh filename="package://cefiro_description/meshes/frame/motor_coupling_1.stl" scale="0.001 0.001 0.001"/>
+      </geometry>
+    </collision>
+  </link>
+  <link name="motor_d3536_mount_1">
+    <inertial>
+      <origin xyz="0.02099976517264429 3.5301522124941975e-07 0.0014999999999999389" rpy="0 0 0"/>
+      <mass value="0.0049294478925385665"/>
+      <inertia ixx="1e-06" iyy="1e-06" izz="1e-06" ixy="0.0" iyz="0.0" ixz="0.0"/>
+    </inertial>
+    <visual>
+      <origin xyz="-0.172706 0.130523 -0.0408" rpy="0 0 0"/>
+      <geometry>
+        <mesh filename="package://cefiro_description/meshes/frame/motor_d3536_mount_1.stl" scale="0.001 0.001 0.001"/>
+      </geometry>
+      <material name="silver"/>
+    </visual>
+    <collision>
+      <origin xyz="-0.172706 0.130523 -0.0408" rpy="0 0 0"/>
+      <geometry>
+        <mesh filename="package://cefiro_description/meshes/frame/motor_d3536_mount_1.stl" scale="0.001 0.001 0.001"/>
+      </geometry>
+    </collision>
+  </link>
+  <link name="motor_d3536_1">
+    <inertial>
+      <origin xyz="0.00311979772526097 -0.00010820481819659444 0.016925643755391226" rpy="0 0 0"/>
+      <mass value="0.09245457976256843"/>
+      <inertia ixx="3e-06" iyy="-1e-06" izz="-9e-06" ixy="-0.000122" iyz="0.0" ixz="-1e-06"/>
+    </inertial>
+    <visual>
+      <origin xyz="-0.193706 0.130523 -0.0438" rpy="0 0 0"/>
+      <geometry>
+        <mesh filename="package://cefiro_description/meshes/frame/motor_d3536_1.stl" scale="0.001 0.001 0.001"/>
+      </geometry>
+      <material name="silver"/>
+    </visual>
+    <collision>
+      <origin xyz="-0.193706 0.130523 -0.0438" rpy="0 0 0"/>
+      <geometry>
+        <mesh filename="package://cefiro_description/meshes/frame/motor_d3536_1.stl" scale="0.001 0.001 0.001"/>
+      </geometry>
+    </collision>
+  </link>
+  <link name="arm_coupling_left__1">
+    <inertial>
+      <origin xyz="-0.01307637591201335 0.006722196062234193 0.01701148304046989" rpy="0 0 0"/>
+      <mass value="0.03789311357416233"/>
+      <inertia ixx="8e-06" iyy="8e-06" izz="9e-06" ixy="-1e-06" iyz="-0.0" ixz="-0.0"/>
+    </inertial>
+    <visual>
+      <origin xyz="-0.027321 0.026359 -0.003" rpy="0 0 0"/>
+      <geometry>
+        <mesh filename="package://cefiro_description/meshes/frame/arm_coupling_left__1.stl" scale="0.001 0.001 0.001"/>
+      </geometry>
+      <material name="silver"/>
+    </visual>
+    <collision>
+      <origin xyz="-0.027321 0.026359 -0.003" rpy="0 0 0"/>
+      <geometry>
+        <mesh filename="package://cefiro_description/meshes/frame/arm_coupling_left__1.stl" scale="0.001 0.001 0.001"/>
+      </geometry>
+    </collision>
+  </link>
+  <link name="propeller_arm__1__1">
+    <inertial>
+      <origin xyz="-0.024571844600186958 -0.024924381030834903 -1.0408340855860843e-17" rpy="0 0 0"/>
+      <mass value="0.01766678419295193"/>
+      <inertia ixx="5e-06" iyy="5e-06" izz="8e-06" ixy="-3e-06" iyz="0.0" ixz="0.0"/>
+    </inertial>
+    <visual>
+      <origin xyz="-0.004348 0.030663 -0.0198" rpy="0 0 0"/>
+      <geometry>
+        <mesh filename="package://cefiro_description/meshes/frame/propeller_arm__1__1.stl" scale="0.001 0.001 0.001"/>
+      </geometry>
+      <material name="silver"/>
+    </visual>
+    <collision>
+      <origin xyz="-0.004348 0.030663 -0.0198" rpy="0 0 0"/>
+      <geometry>
+        <mesh filename="package://cefiro_description/meshes/frame/propeller_arm__1__1.stl" scale="0.001 0.001 0.001"/>
+      </geometry>
+    </collision>
+  </link>
+  <link name="arm-motor_coupling__2__1">
+    <inertial>
+      <origin xyz="-0.005103591280053783 -0.00517646190285577 4.462910728475489e-09" rpy="0 0 0"/>
+      <mass value="0.17482105870117712"/>
+      <inertia ixx="3.3e-05" iyy="3.4e-05" izz="2.9e-05" ixy="4e-06" iyz="-0.0" ixz="0.0"/>
+    </inertial>
+    <visual>
+      <origin xyz="0.044796 0.080512 -0.0198" rpy="0 0 0"/>
+      <geometry>
+        <mesh filename="package://cefiro_description/meshes/frame/arm-motor_coupling__2__1.stl" scale="0.001 0.001 0.001"/>
+      </geometry>
+      <material name="silver"/>
+    </visual>
+    <collision>
+      <origin xyz="0.044796 0.080512 -0.0198" rpy="0 0 0"/>
+      <geometry>
+        <mesh filename="package://cefiro_description/meshes/frame/arm-motor_coupling__2__1.stl" scale="0.001 0.001 0.001"/>
+      </geometry>
+    </collision>
+  </link>
+  <link name="motor_coupling__1__1">
+    <inertial>
+      <origin xyz="-0.024802008214397986 -0.024913127496109855 0.003012980980874668" rpy="0 0 0"/>
+      <mass value="0.08266534784043636"/>
+      <inertia ixx="3.8e-05" iyy="3.7e-05" izz="4.7e-05" ixy="-1.1e-05" iyz="6e-06" ixz="6e-06"/>
+    </inertial>
+    <visual>
+      <origin xyz="0.058837 0.094754 -0.0198" rpy="0 0 0"/>
+      <geometry>
+        <mesh filename="package://cefiro_description/meshes/frame/motor_coupling__1__1.stl" scale="0.001 0.001 0.001"/>
+      </geometry>
+      <material name="silver"/>
+    </visual>
+    <collision>
+      <origin xyz="0.058837 0.094754 -0.0198" rpy="0 0 0"/>
+      <geometry>
+        <mesh filename="package://cefiro_description/meshes/frame/motor_coupling__1__1.stl" scale="0.001 0.001 0.001"/>
+      </geometry>
+    </collision>
+  </link>
+  <link name="motor_d3536_mount__1__1">
+    <inertial>
+      <origin xyz="0.000148897377897389 -0.020999056240172786 0.0015000000000000013" rpy="0 0 0"/>
+      <mass value="0.0049294478925385665"/>
+      <inertia ixx="1e-06" iyy="1e-06" izz="1e-06" ixy="0.0" iyz="0.0" ixz="-0.0"/>
+    </inertial>
+    <visual>
+      <origin xyz="0.095142 0.110429 -0.0408" rpy="0 0 0"/>
+      <geometry>
+        <mesh filename="package://cefiro_description/meshes/frame/motor_d3536_mount__1__1.stl" scale="0.001 0.001 0.001"/>
+      </geometry>
+      <material name="silver"/>
+    </visual>
+    <collision>
+      <origin xyz="0.095142 0.110429 -0.0408" rpy="0 0 0"/>
+      <geometry>
+        <mesh filename="package://cefiro_description/meshes/frame/motor_d3536_mount__1__1.stl" scale="0.001 0.001 0.001"/>
+      </geometry>
+    </collision>
+  </link>
+  <link name="motor_d3536__1__1">
+    <inertial>
+      <origin xyz="0.003120623230976255 -8.641643070833593e-05 0.01692564375539126" rpy="0 0 0"/>
+      <mass value="0.09245457976256843"/>
+      <inertia ixx="5e-06" iyy="-3e-06" izz="-9e-06" ixy="-0.000122" iyz="0.0" ixz="-1e-06"/>
+    </inertial>
+    <visual>
+      <origin xyz="0.094993 0.131428 -0.0438" rpy="0 0 0"/>
+      <geometry>
+        <mesh filename="package://cefiro_description/meshes/frame/motor_d3536__1__1.stl" scale="0.001 0.001 0.001"/>
+      </geometry>
+      <material name="silver"/>
+    </visual>
+    <collision>
+      <origin xyz="0.094993 0.131428 -0.0438" rpy="0 0 0"/>
+      <geometry>
+        <mesh filename="package://cefiro_description/meshes/frame/motor_d3536__1__1.stl" scale="0.001 0.001 0.001"/>
+      </geometry>
+    </collision>
+  </link>
+  <link name="arm_coupling__1__1">
+    <inertial>
+      <origin xyz="-0.013028236068333273 -0.006815018249825833 0.017011481507627036" rpy="0 0 0"/>
+      <mass value="0.0378932947271681"/>
+      <inertia ixx="8e-06" iyy="9e-06" izz="9e-06" ixy="1e-06" iyz="0.0" ixz="-0.0"/>
+    </inertial>
+    <visual>
+      <origin xyz="-0.027321 -0.097359 -0.003" rpy="0 0 0"/>
+      <geometry>
+        <mesh filename="package://cefiro_description/meshes/frame/arm_coupling__1__1.stl" scale="0.001 0.001 0.001"/>
+      </geometry>
+      <material name="silver"/>
+    </visual>
+    <collision>
+      <origin xyz="-0.027321 -0.097359 -0.003" rpy="0 0 0"/>
+      <geometry>
+        <mesh filename="package://cefiro_description/meshes/frame/arm_coupling__1__1.stl" scale="0.001 0.001 0.001"/>
+      </geometry>
+    </collision>
+  </link>
+  <link name="propeller_arm__2__1">
+    <inertial>
+      <origin xyz="-0.024748918536490867 0.024748774643856553 4.85722573273506e-17" rpy="0 0 0"/>
+      <mass value="0.01766678419295193"/>
+      <inertia ixx="5e-06" iyy="5e-06" izz="8e-06" ixy="3e-06" iyz="0.0" ixz="0.0"/>
+    </inertial>
+    <visual>
+      <origin xyz="-0.004351 -0.101467 -0.0198" rpy="0 0 0"/>
+      <geometry>
+        <mesh filename="package://cefiro_description/meshes/frame/propeller_arm__2__1.stl" scale="0.001 0.001 0.001"/>
+      </geometry>
+      <material name="silver"/>
+    </visual>
+    <collision>
+      <origin xyz="-0.004351 -0.101467 -0.0198" rpy="0 0 0"/>
+      <geometry>
+        <mesh filename="package://cefiro_description/meshes/frame/propeller_arm__2__1.stl" scale="0.001 0.001 0.001"/>
+      </geometry>
+    </collision>
+  </link>
+  <link name="arm-motor_coupling__3__1">
+    <inertial>
+      <origin xyz="-0.005140134397008264 0.005139900034449002 4.462910790925534e-09" rpy="0 0 0"/>
+      <mass value="0.17482105870117712"/>
+      <inertia ixx="3.3e-05" iyy="3.3e-05" izz="2.9e-05" ixy="-4e-06" iyz="-0.0" ixz="-0.0"/>
+    </inertial>
+    <visual>
+      <origin xyz="0.045147 -0.150965 -0.0198" rpy="0 0 0"/>
+      <geometry>
+        <mesh filename="package://cefiro_description/meshes/frame/arm-motor_coupling__3__1.stl" scale="0.001 0.001 0.001"/>
+      </geometry>
+      <material name="silver"/>
+    </visual>
+    <collision>
+      <origin xyz="0.045147 -0.150965 -0.0198" rpy="0 0 0"/>
+      <geometry>
+        <mesh filename="package://cefiro_description/meshes/frame/arm-motor_coupling__3__1.stl" scale="0.001 0.001 0.001"/>
+      </geometry>
+    </collision>
+  </link>
+  <link name="motor_coupling__2__1">
+    <inertial>
+      <origin xyz="-0.024735929014131887 0.024978176445044825 0.0030129809808746993" rpy="0 0 0"/>
+      <mass value="0.08266534784043636"/>
+      <inertia ixx="3.7e-05" iyy="3.8e-05" izz="4.7e-05" ixy="1.1e-05" iyz="-6e-06" ixz="6e-06"/>
+    </inertial>
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