Commit message: ✨ New Feature: RViz2 visualization available for CEFIRO's frame, gyro and their assembly

File: cefiro_description/urdf/gyro.xacro (robot description, xacro)
@@ -2,9 +2,8 @@
 <robot name="gyro"
   xmlns:xacro="http://www.ros.org/wiki/xacro">
-  <xacro:include filename="$(find cefiro_description)/urdf/materials.xacro" />
   <link name="base_link">
     <inertial>
-      <origin xyz="0.001157173130374694 -0.014949350635758602 0.021649313649829683" rpy="0 0 0"/>
-      <mass value="0.2961227403148617"/>
+      <origin xyz="0.0011571731303746855 -0.014949350635758592 0.02164931364982968" rpy="0 0 0"/>
+      <mass value="0.2961227403148616"/>
       <inertia ixx="0.000767" iyy="0.00055" izz="0.001242" ixy="0.0" iyz="-0.0" ixz="-0.0"/>
     </inertial>
@@ -12,5 +11,5 @@
       <origin xyz="0 0 0" rpy="0 0 0"/>
       <geometry>
-        <mesh filename="package://cefiro_description/meshes/base_link.stl" scale="0.001 0.001 0.001"/>
+        <mesh filename="package://cefiro_description/meshes/gyro/base_link.stl" scale="0.001 0.001 0.001"/>
       </geometry>
       <material name="silver"/>
@@ -19,5 +18,5 @@
       <origin xyz="0 0 0" rpy="0 0 0"/>
       <geometry>
-        <mesh filename="package://cefiro_description/meshes/base_link.stl" scale="0.001 0.001 0.001"/>
+        <mesh filename="package://cefiro_description/meshes/gyro/base_link.stl" scale="0.001 0.001 0.001"/>
       </geometry>
     </collision>
@@ -32,5 +31,5 @@
       <origin xyz="0.062963 0.098467 -0.017273" rpy="0 0 0"/>
       <geometry>
-        <mesh filename="package://cefiro_description/meshes/gyro_snap-in-leg_1.stl" scale="0.001 0.001 0.001"/>
+        <mesh filename="package://cefiro_description/meshes/gyro/gyro_snap-in-leg_1.stl" scale="0.001 0.001 0.001"/>
       </geometry>
       <material name="silver"/>
@@ -39,5 +38,5 @@
       <origin xyz="0.062963 0.098467 -0.017273" rpy="0 0 0"/>
       <geometry>
-        <mesh filename="package://cefiro_description/meshes/gyro_snap-in-leg_1.stl" scale="0.001 0.001 0.001"/>
+        <mesh filename="package://cefiro_description/meshes/gyro/gyro_snap-in-leg_1.stl" scale="0.001 0.001 0.001"/>
       </geometry>
     </collision>
@@ -52,5 +51,5 @@
       <origin xyz="0.074257 -0.057271 -0.017273" rpy="0 0 0"/>
       <geometry>
-        <mesh filename="package://cefiro_description/meshes/gyro_snap-in-leg__1__1.stl" scale="0.001 0.001 0.001"/>
+        <mesh filename="package://cefiro_description/meshes/gyro/gyro_snap-in-leg__1__1.stl" scale="0.001 0.001 0.001"/>
       </geometry>
       <material name="silver"/>
@@ -59,5 +58,5 @@
       <origin xyz="0.074257 -0.057271 -0.017273" rpy="0 0 0"/>
       <geometry>
-        <mesh filename="package://cefiro_description/meshes/gyro_snap-in-leg__1__1.stl" scale="0.001 0.001 0.001"/>
+        <mesh filename="package://cefiro_description/meshes/gyro/gyro_snap-in-leg__1__1.stl" scale="0.001 0.001 0.001"/>
       </geometry>
     </collision>
@@ -72,5 +71,5 @@
       <origin xyz="-0.065269 -0.068569 -0.017273" rpy="0 0 0"/>
       <geometry>
-        <mesh filename="package://cefiro_description/meshes/gyro_snap-in-leg__2__1.stl" scale="0.001 0.001 0.001"/>
+        <mesh filename="package://cefiro_description/meshes/gyro/gyro_snap-in-leg__2__1.stl" scale="0.001 0.001 0.001"/>
       </geometry>
       <material name="silver"/>
@@ -79,5 +78,5 @@
       <origin xyz="-0.065269 -0.068569 -0.017273" rpy="0 0 0"/>
       <geometry>
-        <mesh filename="package://cefiro_description/meshes/gyro_snap-in-leg__2__1.stl" scale="0.001 0.001 0.001"/>
+        <mesh filename="package://cefiro_description/meshes/gyro/gyro_snap-in-leg__2__1.stl" scale="0.001 0.001 0.001"/>
       </geometry>
     </collision>
@@ -92,5 +91,5 @@
       <origin xyz="-0.074544 0.089198 -0.016523" rpy="0 0 0"/>
       <geometry>
-        <mesh filename="package://cefiro_description/meshes/gyro_snap-in-leg__3__1.stl" scale="0.001 0.001 0.001"/>
+        <mesh filename="package://cefiro_description/meshes/gyro/gyro_snap-in-leg__3__1.stl" scale="0.001 0.001 0.001"/>
       </geometry>
       <material name="silver"/>
@@ -99,5 +98,5 @@
       <origin xyz="-0.074544 0.089198 -0.016523" rpy="0 0 0"/>
       <geometry>
-        <mesh filename="package://cefiro_description/meshes/gyro_snap-in-leg__3__1.stl" scale="0.001 0.001 0.001"/>
+        <mesh filename="package://cefiro_description/meshes/gyro/gyro_snap-in-leg__3__1.stl" scale="0.001 0.001 0.001"/>
       </geometry>
     </collision>
@@ -112,5 +111,5 @@
       <origin xyz="-0.001156 0.014951 -0.031773" rpy="0 0 0"/>
       <geometry>
-        <mesh filename="package://cefiro_description/meshes/gyro_base_CPv12_1.stl" scale="0.001 0.001 0.001"/>
+        <mesh filename="package://cefiro_description/meshes/gyro/gyro_base_CPv12_1.stl" scale="0.001 0.001 0.001"/>
       </geometry>
       <material name="silver"/>
@@ -119,5 +118,5 @@
       <origin xyz="-0.001156 0.014951 -0.031773" rpy="0 0 0"/>
       <geometry>
-        <mesh filename="package://cefiro_description/meshes/gyro_base_CPv12_1.stl" scale="0.001 0.001 0.001"/>
+        <mesh filename="package://cefiro_description/meshes/gyro/gyro_base_CPv12_1.stl" scale="0.001 0.001 0.001"/>
       </geometry>
     </collision>
@@ -132,5 +131,5 @@
       <origin xyz="-0.001156 0.014951 -0.041673" rpy="0 0 0"/>
       <geometry>
-        <mesh filename="package://cefiro_description/meshes/gyro_ccv12_1.stl" scale="0.001 0.001 0.001"/>
+        <mesh filename="package://cefiro_description/meshes/gyro/gyro_ccv12_1.stl" scale="0.001 0.001 0.001"/>
       </geometry>
       <material name="silver"/>
@@ -139,5 +138,5 @@
       <origin xyz="-0.001156 0.014951 -0.041673" rpy="0 0 0"/>
       <geometry>
-        <mesh filename="package://cefiro_description/meshes/gyro_ccv12_1.stl" scale="0.001 0.001 0.001"/>
+        <mesh filename="package://cefiro_description/meshes/gyro/gyro_ccv12_1.stl" scale="0.001 0.001 0.001"/>
       </geometry>
     </collision>
@@ -152,5 +151,5 @@
       <origin xyz="-0.001156 0.014951 -0.059173" rpy="0 0 0"/>
       <geometry>
-        <mesh filename="package://cefiro_description/meshes/gyro_B1P_1.stl" scale="0.001 0.001 0.001"/>
+        <mesh filename="package://cefiro_description/meshes/gyro/gyro_B1P_1.stl" scale="0.001 0.001 0.001"/>
       </geometry>
       <material name="silver"/>
@@ -159,5 +158,5 @@
       <origin xyz="-0.001156 0.014951 -0.059173" rpy="0 0 0"/>
       <geometry>
-        <mesh filename="package://cefiro_description/meshes/gyro_B1P_1.stl" scale="0.001 0.001 0.001"/>
+        <mesh filename="package://cefiro_description/meshes/gyro/gyro_B1P_1.stl" scale="0.001 0.001 0.001"/>
       </geometry>
     </collision>
@@ -165,5 +164,5 @@
   <link name="gyro_Y-DBA_1">
     <inertial>
-      <origin xyz="2.69618244483176e-07 8.605612878756497e-06 0.0022329783234845274" rpy="0 0 0"/>
+      <origin xyz="2.9059467922362865e-07 8.60399398841874e-06 0.0022329783234873724" rpy="0 0 0"/>
       <mass value="0.015293274790880064"/>
       <inertia ixx="6e-06" iyy="6e-06" izz="1.2e-05" ixy="0.0" iyz="-0.0" ixz="-0.0"/>
@@ -172,5 +171,5 @@
       <origin xyz="-0.001156 0.014951 -0.078173" rpy="0 0 0"/>
       <geometry>
-        <mesh filename="package://cefiro_description/meshes/gyro_Y-DBA_1.stl" scale="0.001 0.001 0.001"/>
+        <mesh filename="package://cefiro_description/meshes/gyro/gyro_Y-DBA_1.stl" scale="0.001 0.001 0.001"/>
       </geometry>
       <material name="silver"/>
@@ -179,5 +178,5 @@
       <origin xyz="-0.001156 0.014951 -0.078173" rpy="0 0 0"/>
       <geometry>
-        <mesh filename="package://cefiro_description/meshes/gyro_Y-DBA_1.stl" scale="0.001 0.001 0.001"/>
+        <mesh filename="package://cefiro_description/meshes/gyro/gyro_Y-DBA_1.stl" scale="0.001 0.001 0.001"/>
       </geometry>
     </collision>
@@ -185,5 +184,5 @@
   <link name="gyro_Y-LOCK_1">
     <inertial>
-      <origin xyz="-4.1981279759462087e-07 -4.7087740018096624e-07 -0.005295109629472827" rpy="0 0 0"/>
+      <origin xyz="-4.1981919979804105e-07 -4.708780733560236e-07 -0.005295109629470551" rpy="0 0 0"/>
       <mass value="0.0041583623164599464"/>
       <inertia ixx="0.0" iyy="0.0" izz="0.0" ixy="-0.0" iyz="0.0" ixz="0.0"/>
@@ -192,5 +191,5 @@
       <origin xyz="-0.001156 0.014951 -0.082473" rpy="0 0 0"/>
       <geometry>
-        <mesh filename="package://cefiro_description/meshes/gyro_Y-LOCK_1.stl" scale="0.001 0.001 0.001"/>
+        <mesh filename="package://cefiro_description/meshes/gyro/gyro_Y-LOCK_1.stl" scale="0.001 0.001 0.001"/>
       </geometry>
       <material name="silver"/>
@@ -199,5 +198,5 @@
       <origin xyz="-0.001156 0.014951 -0.082473" rpy="0 0 0"/>
       <geometry>
-        <mesh filename="package://cefiro_description/meshes/gyro_Y-LOCK_1.stl" scale="0.001 0.001 0.001"/>
+        <mesh filename="package://cefiro_description/meshes/gyro/gyro_Y-LOCK_1.stl" scale="0.001 0.001 0.001"/>
       </geometry>
     </collision>
@@ -205,19 +204,19 @@
   <link name="gyro_CON-Y_368mm_1">
     <inertial>
-      <origin xyz="0.00015725718637999244 0.13082811230823058 0.13105552856831715" rpy="0 0 0"/>
+      <origin xyz="0.00046014841241998647 0.1308280219229364 0.13105552856890101" rpy="0 0 0"/>
       <mass value="0.07094391733872507"/>
-      <inertia ixx="0.000807" iyy="0.000404" izz="0.000405" ixy="-0.0" iyz="-0.000403" ixz="0.0"/>
-    </inertial>
-    <visual>
-      <origin xyz="-0.001156 -0.125802 -0.086526" rpy="0 0 0"/>
-      <geometry>
-        <mesh filename="package://cefiro_description/meshes/gyro_CON-Y_368mm_1.stl" scale="0.001 0.001 0.001"/>
-      </geometry>
-      <material name="silver"/>
-    </visual>
-    <collision>
-      <origin xyz="-0.001156 -0.125802 -0.086526" rpy="0 0 0"/>
-      <geometry>
-        <mesh filename="package://cefiro_description/meshes/gyro_CON-Y_368mm_1.stl" scale="0.001 0.001 0.001"/>
+      <inertia ixx="0.000807" iyy="0.000404" izz="0.000405" ixy="-1e-06" iyz="-0.000403" ixz="-1e-06"/>
+    </inertial>
+    <visual>
+      <origin xyz="-0.001481 -0.125801 -0.086526" rpy="0 0 0"/>
+      <geometry>
+        <mesh filename="package://cefiro_description/meshes/gyro/gyro_CON-Y_368mm_1.stl" scale="0.001 0.001 0.001"/>
+      </geometry>
+      <material name="silver"/>
+    </visual>
+    <collision>
+      <origin xyz="-0.001481 -0.125801 -0.086526" rpy="0 0 0"/>
+      <geometry>
+        <mesh filename="package://cefiro_description/meshes/gyro/gyro_CON-Y_368mm_1.stl" scale="0.001 0.001 0.001"/>
       </geometry>
     </collision>
@@ -225,19 +224,39 @@
   <link name="gyro_CON-Y_368mm__1__1">
     <inertial>
-      <origin xyz="0.00015725718260796982 -0.13105536657572212 0.13082819543817187" rpy="0 0 0"/>
+      <origin xyz="-0.0001451604414352285 -0.13105600467752276 0.1308281954375885" rpy="0 0 0"/>
       <mass value="0.07094391733872507"/>
-      <inertia ixx="0.000807" iyy="0.000405" izz="0.000404" ixy="-0.0" iyz="0.000403" ixz="-0.0"/>
-    </inertial>
-    <visual>
-      <origin xyz="-0.001156 0.155705 -0.086526" rpy="0 0 0"/>
-      <geometry>
-        <mesh filename="package://cefiro_description/meshes/gyro_CON-Y_368mm__1__1.stl" scale="0.001 0.001 0.001"/>
-      </geometry>
-      <material name="silver"/>
-    </visual>
-    <collision>
-      <origin xyz="-0.001156 0.155705 -0.086526" rpy="0 0 0"/>
-      <geometry>
-        <mesh filename="package://cefiro_description/meshes/gyro_CON-Y_368mm__1__1.stl" scale="0.001 0.001 0.001"/>
+      <inertia ixx="0.000807" iyy="0.000405" izz="0.000404" ixy="-1e-06" iyz="0.000403" ixz="1e-06"/>
+    </inertial>
+    <visual>
+      <origin xyz="-0.00083 0.155704 -0.086526" rpy="0 0 0"/>
+      <geometry>
+        <mesh filename="package://cefiro_description/meshes/gyro/gyro_CON-Y_368mm__1__1.stl" scale="0.001 0.001 0.001"/>
+      </geometry>
+      <material name="silver"/>
+    </visual>
+    <collision>
+      <origin xyz="-0.00083 0.155704 -0.086526" rpy="0 0 0"/>
+      <geometry>
+        <mesh filename="package://cefiro_description/meshes/gyro/gyro_CON-Y_368mm__1__1.stl" scale="0.001 0.001 0.001"/>
+      </geometry>
+    </collision>
+  </link>
+  <link name="gyro_B2S-R_1">
+    <inertial>
+      <origin xyz="-0.000225 0.417397 -0.348219" rpy="0 0 0"/>
+      <mass value="0.0"/>
+      <inertia ixx="0.0" iyy="0.0" izz="0.0" ixy="0.0" iyz="0.0" ixz="0.0"/>
+    </inertial>
+    <visual>
+      <origin xyz="-0.000225 0.417397 -0.348219" rpy="0 0 0"/>
+      <geometry>
+        <mesh filename="package://cefiro_description/meshes/gyro/gyro_B2S-R_1.stl" scale="0.001 0.001 0.001"/>
+      </geometry>
+      <material name="silver"/>
+    </visual>
+    <collision>
+      <origin xyz="-0.000225 0.417397 -0.348219" rpy="0 0 0"/>
+      <geometry>
+        <mesh filename="package://cefiro_description/meshes/gyro/gyro_B2S-R_1.stl" scale="0.001 0.001 0.001"/>
       </geometry>
     </collision>
@@ -245,39 +264,19 @@
   <link name="gyro_B2S_1">
     <inertial>
-      <origin xyz="-0.001156 -0.387495 -0.348219" rpy="0 0 0"/>
-      <mass value="0.0"/>
-      <inertia ixx="0.0" iyy="0.0" izz="0.0" ixy="0.0" iyz="0.0" ixz="0.0"/>
-    </inertial>
-    <visual>
-      <origin xyz="-0.001156 -0.387495 -0.348219" rpy="0 0 0"/>
-      <geometry>
-        <mesh filename="package://cefiro_description/meshes/gyro_B2S_1.stl" scale="0.001 0.001 0.001"/>
-      </geometry>
-      <material name="silver"/>
-    </visual>
-    <collision>
-      <origin xyz="-0.001156 -0.387495 -0.348219" rpy="0 0 0"/>
-      <geometry>
-        <mesh filename="package://cefiro_description/meshes/gyro_B2S_1.stl" scale="0.001 0.001 0.001"/>
-      </geometry>
-    </collision>
-  </link>
-  <link name="gyro_B2S-R_1">
-    <inertial>
-      <origin xyz="-0.001156 0.417398 -0.348219" rpy="0 0 0"/>
-      <mass value="0.0"/>
-      <inertia ixx="0.0" iyy="0.0" izz="0.0" ixy="0.0" iyz="0.0" ixz="0.0"/>
-    </inertial>
-    <visual>
-      <origin xyz="-0.001156 0.417398 -0.348219" rpy="0 0 0"/>
-      <geometry>
-        <mesh filename="package://cefiro_description/meshes/gyro_B2S-R_1.stl" scale="0.001 0.001 0.001"/>
-      </geometry>
-      <material name="silver"/>
-    </visual>
-    <collision>
-      <origin xyz="-0.001156 0.417398 -0.348219" rpy="0 0 0"/>
-      <geometry>
-        <mesh filename="package://cefiro_description/meshes/gyro_B2S-R_1.stl" scale="0.001 0.001 0.001"/>
+      <origin xyz="-0.002086 -0.387494 -0.348219" rpy="0 0 0"/>
+      <mass value="0.0"/>
+      <inertia ixx="0.0" iyy="0.0" izz="0.0" ixy="0.0" iyz="0.0" ixz="0.0"/>
+    </inertial>
+    <visual>
+      <origin xyz="-0.002086 -0.387494 -0.348219" rpy="0 0 0"/>
+      <geometry>
+        <mesh filename="package://cefiro_description/meshes/gyro/gyro_B2S_1.stl" scale="0.001 0.001 0.001"/>
+      </geometry>
+      <material name="silver"/>
+    </visual>
+    <collision>
+      <origin xyz="-0.002086 -0.387494 -0.348219" rpy="0 0 0"/>
+      <geometry>
+        <mesh filename="package://cefiro_description/meshes/gyro/gyro_B2S_1.stl" scale="0.001 0.001 0.001"/>
       </geometry>
     </collision>
@@ -285,19 +284,19 @@
   <link name="gyro_A2-LW_1">
     <inertial>
-      <origin xyz="0.098057 -0.458094 -0.418818" rpy="0 0 0"/>
-      <mass value="0.0"/>
-      <inertia ixx="0.0" iyy="0.0" izz="0.0" ixy="0.0" iyz="0.0" ixz="0.0"/>
-    </inertial>
-    <visual>
-      <origin xyz="0.098057 -0.458094 -0.418818" rpy="0 0 0"/>
-      <geometry>
-        <mesh filename="package://cefiro_description/meshes/gyro_A2-LW_1.stl" scale="0.001 0.001 0.001"/>
-      </geometry>
-      <material name="silver"/>
-    </visual>
-    <collision>
-      <origin xyz="0.098057 -0.458094 -0.418818" rpy="0 0 0"/>
-      <geometry>
-        <mesh filename="package://cefiro_description/meshes/gyro_A2-LW_1.stl" scale="0.001 0.001 0.001"/>
+      <origin xyz="-0.002089 -0.388847 -0.488972" rpy="0 0 0"/>
+      <mass value="0.0"/>
+      <inertia ixx="0.0" iyy="0.0" izz="0.0" ixy="0.0" iyz="0.0" ixz="0.0"/>
+    </inertial>
+    <visual>
+      <origin xyz="-0.002089 -0.388847 -0.488972" rpy="0 0 0"/>
+      <geometry>
+        <mesh filename="package://cefiro_description/meshes/gyro/gyro_A2-LW_1.stl" scale="0.001 0.001 0.001"/>
+      </geometry>
+      <material name="silver"/>
+    </visual>
+    <collision>
+      <origin xyz="-0.002089 -0.388847 -0.488972" rpy="0 0 0"/>
+      <geometry>
+        <mesh filename="package://cefiro_description/meshes/gyro/gyro_A2-LW_1.stl" scale="0.001 0.001 0.001"/>
       </geometry>
     </collision>
@@ -305,19 +304,19 @@
   <link name="gyro_CON-P_360mm_1">
     <inertial>
-      <origin xyz="-0.1802061546651206 -0.0001503950917337571 0.0001782116110824461" rpy="0 0 0"/>
+      <origin xyz="0.12691013516768695 -0.1275268308090541 -0.00012374419014998805" rpy="0 0 0"/>
       <mass value="0.0670222866413884"/>
-      <inertia ixx="2e-06" iyy="0.000722" izz="0.000722" ixy="-0.0" iyz="0.0" ixz="-0.0"/>
-    </inertial>
-    <visual>
-      <origin xyz="0.217878 -0.502904 -0.463796" rpy="0 0 0"/>
-      <geometry>
-        <mesh filename="package://cefiro_description/meshes/gyro_CON-P_360mm_1.stl" scale="0.001 0.001 0.001"/>
-      </geometry>
-      <material name="silver"/>
-    </visual>
-    <collision>
-      <origin xyz="0.217878 -0.502904 -0.463796" rpy="0 0 0"/>
-      <geometry>
-        <mesh filename="package://cefiro_description/meshes/gyro_CON-P_360mm_1.stl" scale="0.001 0.001 0.001"/>
+      <inertia ixx="0.000364" iyy="0.00036" izz="0.000722" ixy="0.00036" iyz="0.0" ixz="-0.0"/>
+    </inertial>
+    <visual>
+      <origin xyz="-0.118665 -0.362637 -0.489072" rpy="0 0 0"/>
+      <geometry>
+        <mesh filename="package://cefiro_description/meshes/gyro/gyro_CON-P_360mm_1.stl" scale="0.001 0.001 0.001"/>
+      </geometry>
+      <material name="silver"/>
+    </visual>
+    <collision>
+      <origin xyz="-0.118665 -0.362637 -0.489072" rpy="0 0 0"/>
+      <geometry>
+        <mesh filename="package://cefiro_description/meshes/gyro/gyro_CON-P_360mm_1.stl" scale="0.001 0.001 0.001"/>
       </geometry>
     </collision>
@@ -325,19 +324,239 @@
   <link name="gyro_A1-LW_1">
     <inertial>
-      <origin xyz="0.577998 -0.502904 -0.463796" rpy="0 0 0"/>
-      <mass value="0.0"/>
-      <inertia ixx="0.0" iyy="0.0" izz="0.0" ixy="0.0" iyz="0.0" ixz="0.0"/>
-    </inertial>
-    <visual>
-      <origin xyz="0.577998 -0.502904 -0.463796" rpy="0 0 0"/>
-      <geometry>
-        <mesh filename="package://cefiro_description/meshes/gyro_A1-LW_1.stl" scale="0.001 0.001 0.001"/>
-      </geometry>
-      <material name="silver"/>
-    </visual>
-    <collision>
-      <origin xyz="0.577998 -0.502904 -0.463796" rpy="0 0 0"/>
-      <geometry>
-        <mesh filename="package://cefiro_description/meshes/gyro_A1-LW_1.stl" scale="0.001 0.001 0.001"/>
+      <origin xyz="-0.372719 -0.107405 -0.48929" rpy="0 0 0"/>
+      <mass value="0.0"/>
+      <inertia ixx="0.0" iyy="0.0" izz="0.0" ixy="0.0" iyz="0.0" ixz="0.0"/>
+    </inertial>
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